File: kicad/kicad_sensor_on_side_big_display.kicad_pcb (KiCad board)
At the start: 2 copper layers, 26.5 x 42.5 mm, 12 parts, among them SW1 SW_Push, SW2 SW_Push, U1 nice_nano, U2 GY-BNO08X, U3 SSD1306_OLED_042

Commit message: kicad: fix project refs
Parts:
- added U4: SSD1306_OLED_042, Connector_PinHeader_2.54mm:PinHeader_1x04_P2.54mm_Vertical, F.Cu at (172.5, 62.6)
- moved SW_POWER1 0.50 mm to (195.0, 47.5)
Routing:
- net Net-(U1-VCC): track 40.9 -> 39.1 mm
Other:
- board size 26.5 x 42.5 mm -> 47.6 x 44.9 mm
