File: kicad/v2_sensor_on_side/v2_sensor_on_side.kicad_sch (KiCad schematic)
At the start: 9 parts, among them SW1 SW_Push, SW2 SW_Push, U1 nice_nano, U2 GY-BNO08X, U3 SSD1306_OLED_042, U4 SSD1306_OLED_042

Commit message: kicad: tidy up
Parts:
- removed U4: SSD1306_OLED_042, Connector_PinHeader_2.54mm:PinHeader_1x04_P2.54mm_Vertical, symbol knife_level:SSD1306_OLED_042
