File: kicad/v4_fully_integrated_pc/v4_fully_integrated_pc.kicad_sch (KiCad schematic)
At the start: 18 parts, among them SW1 SW_Push, SW2 SW_Push, U1 nice_nano, U3 SSD1306_OLED_042, U4 SSD1306_OLED_042

Commit message: before ref
Parts:
- renumbered BAT+1 to B+1, BAT-1 to B-1
Changed lines of the file:
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@@
 		(dnp no)
 		(fields_autoplaced yes)
-		(property "Reference" "BAT+1"
+		(property "Reference" "B+1"
 			(at 537.21 88.8999 0)
 			(show_name no)
@@
 			(project "v4_fully_integrated_pc"
 				(path "/8b17f9a6-b000-4ccb-b0d9-cb9857b67250"
-					(reference "BAT+1")
+					(reference "B+1")
 					(unit 1)
 				)
@@
 		(dnp no)
 		(fields_autoplaced yes)
-		(property "Reference" "BAT-1"
+		(property "Reference" "B-1"
 			(at 453.39 81.28 0)
 			(show_name no)
@@
 			(project "v4_fully_integrated_pc"
 				(path "/8b17f9a6-b000-4ccb-b0d9-cb9857b67250"
-					(reference "BAT-1")
-					(unit 1)
-				)
+					(reference "B-1")
+					(unit 1)
+				)

Commit message: fix calculation to be more tolerant to spinning
Parts:
- renumbered BNO085 to U2
Changed lines of the file:
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@@
 		(dnp no)
 		(fields_autoplaced yes)
-		(property "Reference" "BNO085"
+		(property "Reference" "U2"
 			(at 361.95 81.28 0)
 			(show_name no)
@@
 			(project "v4_fully_integrated_pc"
 				(path "/8b17f9a6-b000-4ccb-b0d9-cb9857b67250"
-					(reference "BNO085")
+					(reference "U2")
 					(unit 1)
 				)
